File: Hardware/TestingRig/_autosave-TestingRig.kicad_sch (KiCad schematic)
At the start: 66 parts, among them J1 Conn_01x04_Pin, J2 Conn_01x04_Pin, J3 Conn_01x04_Pin, J4 Conn_01x04_Pin, J5 Conn_01x04_Pin, J6 Conn_01x04_Pin

Commit message: message
Parts:
- removed C2 (x3): 100n, Capacitor_SMD:C_0603_1608Metric, symbol Device:C_Small
- removed D10, D20, D30: WS2812, LED_SMD:LED_WS2812_PLCC6_5.0x5.0mm_P1.6mm, symbol LED:WS2812
- renumbered D11 to D10, D12 to D11, D13 to D12, D14 to D13, D15 to D14, D16 to D15, D17 to D16, D18 to D17, D19 to D18, D21 to D19, D22 to D20, D23 to D21, D24 to D22, D25 to D23, D26 to D24, D27 to D25, D28 to D26, D29 to D27
Connections:
- net Dout10 is gone; now on net Dout9: J2.2 (Pin_2)
- net Dout19 is gone; now on net Dout18: D18.1 (DOUT)
- net Dout20 is gone; now on net Dout18: J4.2 (Pin_2)
- net Dout29 is gone; now on net Dout27: D27.1 (DOUT)
- net Dout30 is gone; now on net Dout27: J6.2 (Pin_2)
- net Dout18: no longer D17.1 (DOUT), D18.2 (DIN)
- net Dout27: no longer D25.1 (DOUT), D26.2 (DIN)
- net Din11 renamed Din10
- net Din21 renamed Din19
- net Dout12: no longer names the net of D11.1 (DOUT), D12.2 (DIN)
- net Dout13: no longer names the net of D12.1 (DOUT), D13.2 (DIN)
- net Dout14: no longer names the net of D13.1 (DOUT), D14.2 (DIN)
- net Dout15: no longer names the net of D14.1 (DOUT), D15.2 (DIN)
- net Dout16: no longer names the net of D15.1 (DOUT), D16.2 (DIN)
- net Dout17: no longer names the net of D16.1 (DOUT), D17.2 (DIN)
- net Dout2: no longer names the net of D2.1 (DOUT), D3.2 (DIN)
- net Dout22: no longer names the net of D20.1 (DOUT), D21.2 (DIN)
- net Dout23: no longer names the net of D21.1 (DOUT), D22.2 (DIN)
- net Dout24: no longer names the net of D22.1 (DOUT), D23.2 (DIN)
- net Dout25: no longer names the net of D23.1 (DOUT), D24.2 (DIN)
- net Dout26: no longer names the net of D24.1 (DOUT), D25.2 (DIN)
- net Dout28: no longer names the net of D26.1 (DOUT), D27.2 (DIN)
- net Dout3: no longer names the net of D3.1 (DOUT), D4.2 (DIN)
- net Dout4: no longer names the net of D4.1 (DOUT), D5.2 (DIN)
- net Dout5: no longer names the net of D5.1 (DOUT), D6.2 (DIN)
- net Dout6: no longer names the net of D6.1 (DOUT), D7.2 (DIN)
- net Dout7: no longer names the net of D7.1 (DOUT), D8.2 (DIN)
- net Dout8: no longer names the net of D8.1 (DOUT), D9.2 (DIN)
- new net: D25.1 (DOUT), D26.2 (DIN)
- new net: D17.1 (DOUT), D18.2 (DIN)
Other:
- moved on the sheet: J1, J2, J3, J4, J5, J6
