File: Hardware/TestingRig/TestingRig.kicad_pcb (KiCad board)
At the start: 2 copper layers, 100 x 100 mm, 60 parts, among them J1 Conn_01x04_Pin, J2 Conn_01x04_Pin, J3 Conn_01x04_Pin, J4 Conn_01x04_Pin, J5 Conn_01x04_Pin, J6 Conn_01x04_Pin

Commit message: $1
Changed lines of the file:
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@@
     (property "ki_description" "Generic connector, single row, 01x04, script generated")
     (property "ki_keywords" "connector")
-    (attr through_hole)
+    (attr through_hole exclude_from_bom)
     (fp_text reference "J3" (at 0 -2.33) (layer "F.SilkS")
         (effects (font (size 1 1) (thickness 0.15)))
@@
     (property "ki_description" "Generic connector, single row, 01x04, script generated")
     (property "ki_keywords" "connector")
-    (attr through_hole)
+    (attr through_hole exclude_from_bom)
     (fp_text reference "J2" (at 0 -2.33) (layer "F.SilkS")
         (effects (font (size 1 1) (thickness 0.15)))
@@
     (property "ki_description" "Generic connector, single row, 01x04, script generated")
     (property "ki_keywords" "connector")
-    (attr through_hole)
+    (attr through_hole exclude_from_bom)
     (fp_text reference "J6" (at 0 -2.33) (layer "F.SilkS")
         (effects (font (size 1 1) (thickness 0.15)))
@@
     (property "ki_description" "Generic connector, single row, 01x04, script generated")
     (property "ki_keywords" "connector")
-    (attr through_hole)
+    (attr through_hole exclude_from_bom)
     (fp_text reference "J1" (at 0 -2.33) (layer "F.SilkS")
         (effects (font (size 1 1) (thickness 0.15)))
@@
     (property "ki_description" "Generic connector, single row, 01x04, script generated")
     (property "ki_keywords" "connector")
-    (attr through_hole)
+    (attr through_hole exclude_from_bom)
     (fp_text reference "J5" (at 0 -2.33) (layer "F.SilkS")
         (effects (font (size 1 1) (thickness 0.15)))
@@
     (property "ki_description" "Generic connector, single row, 01x04, script generated")
     (property "ki_keywords" "connector")
-    (attr through_hole)
+    (attr through_hole exclude_from_bom)
     (fp_text reference "J4" (at 0 -2.33) (layer "F.SilkS")
         (effects (font (size 1 1) (thickness 0.15)))
@@
   (gr_line locked (start 190 150.75) (end 94 150.75)
     (stroke (width 0.1) (type default)) (layer "Edge.Cuts"))
-  (gr_rect (start 220 62) (end 312 154)
+  (gr_rect (start 92 50.7) (end 96 54.7)
+    (stroke (width 0.15) (type default)) (fill none) (layer "User.1"))
+  (gr_rect (start 188 146.75) (end 192 150.75)
+    (stroke (width 0.15) (type default)) (fill none) (layer "User.1"))
+  (gr_rect (start 92 146.75) (end 96 150.75)
+    (stroke (width 0.15) (type default)) (fill none) (layer "User.1"))
+  (gr_rect (start 188 50.75) (end 192 54.75)
     (stroke (width 0.15) (type default)) (fill none) (layer "User.1"))
   (gr_text "Din" (at 98.2 64.7) (layer "F.SilkS")
@@
     (effects (font (size 1 1) (thickness 0.15)) (justify left bottom))
   )
-  (via locked (at 188 54) (size 3) (drill 2.2) (layers "F.Cu" "B.Cu") (free) (net 0))
-  (via locked (at 188 146) (size 3) (drill 2.2) (layers "F.Cu" "B.Cu") (free) (net 0))
-  (via locked (at 96 54) (size 3) (drill 2.2) (layers "F.Cu" "B.Cu") (free) (net 0))
-  (via locked (at 96 146) (size 3) (drill 2.2) (layers "F.Cu" "B.Cu") (free) (net 0))
+  (dimension (type aligned) (layer "User.1")
+    (pts (xy 96 146.75) (xy 188 146.75))
+    (height 16.949999)
+    (gr_text "92.0000 mm" (at 142 162.549999) (layer "User.1")
+      (effects (font (size 1 1) (thickness 0.15)))
+    )
+    (format (prefix "") (suffix "") (units 3) (units_format 1) (precision 4))
+    (style (thickness 0.15) (arrow_length 1.27) (text_position_mode 0) (extension_height 0.58642) (extension_offset 0.5) keep_text_aligned)
+  )
+  (dimension (type aligned) (layer "User.1")
+    (pts (xy 96 146.75) (xy 92 146.75))
+    (height -17)
+    (gr_text "4.0000 mm" (at 94 162.6) (layer "User.1")
+      (effects (font (size 1 1) (thickness 0.15)))
+    )
+    (format (prefix "") (suffix "") (units 3) (units_format 1) (precision 4))
+    (style (thickness 0.15) (arrow_length 1.27) (text_position_mode 0) (extension_height 0.58642) (extension_offset 0.5) keep_text_aligned)
+  )
+  (dimension (type aligned) (layer "User.1")
+    (pts (xy 92 146.75) (xy 192 146.75))
+    (height 23.599999)
+    (gr_text "100.0000 mm" (at 142 169.199999) (layer "User.1")
+      (effects (font (size 1 1) (thickness 0.15)))
+    )
+    (format (prefix "") (suffix "") (units 3) (units_format 1) (precision 4))
+    (style (thickness 0.15) (arrow_length 1.27) (text_position_mode 0) (extension_height 0.58642) (extension_offset 0.5) keep_text_aligned)
+  )
+  (dimension (type aligned) (layer "User.1")
+    (pts (xy 188 150.75) (xy 188 146.75))
+    (height 7.7)
+    (gr_text "4.0000 mm" (at 194.55 148.75 90) (layer "User.1")
+      (effects (font (size 1 1) (thickness 0.15)))
+    )
+    (format (prefix "") (suffix "") (units 3) (units_format 1) (precision 4))
+    (style (thickness 0.15) (arrow_length 1.27) (text_position_mode 0) (extension_height 0.58642) (extension_offset 0.5) keep_text_aligned)
+  )
+  (dimension (type aligned) (layer "User.1")
+    (pts (xy 188 146.75) (xy 192 146.75))
+    (height 16.9)
+    (gr_text "4.0000 mm" (at 190 162.5) (layer "User.1")
+      (effects (font (size 1 1) (thickness 0.15)))
+    )
+    (format (prefix "") (suffix "") (units 3) (units_format 1) (precision 4))
+    (style (thickness 0.15) (arrow_length 1.27) (text_position_mode 0) (extension_height 0.58642) (extension_offset 0.5) keep_text_aligned)
+  )
+  (dimension (type aligned) (layer "User.1")
+    (pts (xy 96 150.75) (xy 96 146.75))
+    (height -6.2)
+    (gr_text "4.0000 mm" (at 88.65 148.75 90) (layer "User.1")
+      (effects (font (size 1 1) (thickness 0.15)))
+    )
+    (format (prefix "") (suffix "") (units 3) (units_format 1) (precision 4))
+    (style (thickness 0.15) (arrow_length 1.27) (text_position_mode 0) (extension_height 0.58642) (extension_offset 0.5) keep_text_aligned)
+  )
+  (via locked (at 188 54.75) (size 3) (drill 2.2) (layers "F.Cu" "B.Cu") (free) (net 0))
+  (via locked (at 188 146.75) (size 3) (drill 2.2) (layers "F.Cu" "B.Cu") (free) (net 0))
+  (via locked (at 96 54.75) (size 3) (drill 2.2) (layers "F.Cu" "B.Cu") (free) (net 0))
+  (via locked (at 96 146.75) (size 3) (drill 2.2) (layers "F.Cu" "B.Cu") (free) (net 0))
   (segment (start 158.593125 131.448563) (end 158.623869 131.417819) (width 0.25) (layer "F.Cu") (net 1))
   (segment (start 122.570382 100.192968) (end 122.570382 95.410716) (width 0.25) (layer "F.Cu") (net 1))
@@
   (via (at 113.734881 59.400957) (size 0.8) (drill 0.4) (layers "F.Cu" "B.Cu") (free) (net 1))
   (via (at 140.617371 131.417819) (size 0.8) (drill 0.4) (layers "F.Cu" "B.Cu") (free) (net 1))
-  (segment locked (start 94.625 99.34) (end 94.525 99.44) (width 0.3) (layer "F.Cu") (net 2))
+  (segment (start 94.625 99.34) (end 94.525 99.44) (width 0.3) (layer "F.Cu") (net 2))
   (segment (start 106.143125 142.917819) (end 108.504375 142.917819) (width 0.3) (layer "F.Cu") (net 3))
   (segment (start 111.504375 139.917819) (end 114.343125 139.917819) (width 0.3) (layer "F.Cu") (net 3))
@@
   (segment (start 171.631632 70.900957) (end 174.631632 67.900957) (width 0.3) (layer "F.Cu") (net 59))
   (segment (start 167.720382 69.100957) (end 167.720382 69.350957) (width 0.3) (layer "F.Cu") (net 59))
-  (zone locked (net 2) (net_name "/+5V") (layer "F.Cu") (hatch edge 0.5)
+  (zone (net 2) (net_name "/+5V") (layer "F.Cu") (hatch edge 0.5)
     (connect_pads (clearance 0.5))
     (min_thickness 0.25) (filled_areas_thickness no)
@@
     )
   )
-  (zone locked (net 1) (net_name "GND") (layer "B.Cu") (hatch edge 0.5)
+  (zone (net 1) (net_name "GND") (layer "B.Cu") (hatch edge 0.5)
     (priority 1)
     (connect_pads (clearance 0.5))
@@
     )
   )
-  (group "" locked (id 34c8e807-0276-4a90-b096-0a279491e70d)
-    (members
-      02617bbb-1821-4c11-8934-8f3d552dabe7
-      3fea7d6f-605d-4968-ace8-d39164eaf8c3
-      d8c8c078-f829-4a96-a612-d4918d61bc11
-      dae42bb6-094e-4e61-b837-d4ed804aae5f
-      e1def061-d1ca-4224-87e6-fa5387032979
-    )
-  )

Commit message: message
Parts:
- added G***: LOGO, LOGO, B.Cu at (180.3, 119.1)
