File: Hardware/TestingRig/TestingRig.kicad_pcb (KiCad board)
At the start: 2 copper layers, 100 x 100 mm, 61 parts, among them J1 Conn_01x04_Pin, J2 Conn_01x04_Pin, J3 Conn_01x04_Pin, J4 Conn_01x04_Pin, J5 Conn_01x04_Pin, J6 Conn_01x04_Pin

Commit message: $1
Parts:
- G***: moved to F.Cu
- turned G*** to 0 degrees

Commit message: message
Parts:
- D1, D10, D11, D12, D13, D14, D15, D16, D17, D18, D19, D2, D20, D21, D22, D23, D24, D25, D26, D27, D3, D4, D5, D6, D7, D8, D9: footprint LED_SMD:LED_WS2812_PLCC6_5.0x5.0mm_P1.6mm -> LED_SMD:LED_WS2812B_PLCC4_5.0x5.0mm_P3.2mm
- moved C1 13.6 mm to (104.6, 145.7), turned to 90 degrees
- moved C2 13.6 mm to (113.6, 145.7), turned to 90 degrees
- moved C3 13.6 mm to (122.6, 145.7), turned to 90 degrees
- moved C4 13.6 mm to (131.6, 145.7), turned to 90 degrees
- moved C5 13.6 mm to (140.6, 145.7), turned to 90 degrees
- moved C6 13.6 mm to (149.6, 145.7), turned to 90 degrees
- moved C7 13.6 mm to (158.6, 145.7), turned to 90 degrees
- moved C8 13.6 mm to (167.6, 145.7), turned to 90 degrees
- moved C9 13.6 mm to (176.6, 145.7), turned to 90 degrees
- moved C14 13.5 mm to (131.7, 109.7), turned to 90 degrees
- moved C15 13.5 mm to (140.7, 109.7), turned to 90 degrees
- moved C16 13.5 mm to (149.7, 109.7), turned to 90 degrees
- moved C17 13.5 mm to (158.7, 109.7), turned to 90 degrees
- moved C18 13.5 mm to (167.7, 109.7), turned to 90 degrees
- moved C19 13.5 mm to (176.7, 109.7), turned to 90 degrees
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- renumbered C10 to C11, C11 to C12, C12 to C13, C13 to C14, C14 to C15, C15 to C16, C16 to C17, C17 to C18, C18 to C19, C19 to C21, C20 to C22, C21 to C23, C22 to C24, C23 to C25, C24 to C26, C25 to C27, C26 to C28, C27 to C29, J5 to J1, J6 to J2, J1 to J3, J2 to J4, J3 to J5, J4 to J6
Connections:
- D1 pad 1: /Dout1 -> /+5V
- D1 pad 2: /Din1 -> /Dout1
- D1 pad 3: /+5V -> GND
- D1 pad 4: unconnected-(D1-NC-Pad4) -> /Din1
- D10 pad 1: /Dout11 -> /+5V
- D10 pad 2: /Din10 -> /Dout11
- D10 pad 3: /+5V -> GND
- D10 pad 4: unconnected-(D10-NC-Pad4) -> /Din10
- D11 pad 1: Net-(D11-DOUT) -> /+5V
- D11 pad 2: /Dout11 -> Net-(D11-DOUT)
- D11 pad 3: /+5V -> GND
- D11 pad 4: unconnected-(D11-NC-Pad4) -> /Dout11
- D12 pad 1: Net-(D12-DOUT) -> /+5V
- D12 pad 2: Net-(D11-DOUT) -> Net-(D12-DOUT)
- D12 pad 3: /+5V -> GND
- D12 pad 4: unconnected-(D12-NC-Pad4) -> Net-(D11-DOUT)
- D13 pad 1: Net-(D13-DOUT) -> /+5V
- D13 pad 2: Net-(D12-DOUT) -> Net-(D13-DOUT)
- D13 pad 3: /+5V -> GND
- D13 pad 4: unconnected-(D13-NC-Pad4) -> Net-(D12-DOUT)
- D14 pad 1: Net-(D14-DOUT) -> /+5V
- D14 pad 2: Net-(D13-DOUT) -> Net-(D14-DOUT)
- D14 pad 3: /+5V -> GND
- D14 pad 4: unconnected-(D14-NC-Pad4) -> Net-(D13-DOUT)
- D15 pad 1: Net-(D15-DOUT) -> /+5V
- D15 pad 2: Net-(D14-DOUT) -> Net-(D15-DOUT)
- D15 pad 3: /+5V -> GND
- D15 pad 4: unconnected-(D15-NC-Pad4) -> Net-(D14-DOUT)
- D16 pad 1: Net-(D16-DOUT) -> /+5V
- D16 pad 2: Net-(D15-DOUT) -> Net-(D16-DOUT)
- D16 pad 3: /+5V -> GND
- D16 pad 4: unconnected-(D16-NC-Pad4) -> Net-(D15-DOUT)
- D17 pad 1: Net-(D17-DOUT) -> /+5V
- D17 pad 2: Net-(D16-DOUT) -> Net-(D17-DOUT)
- D17 pad 3: /+5V -> GND
- D17 pad 4: unconnected-(D17-NC-Pad4) -> Net-(D16-DOUT)
- D18 pad 1: /Dout18 -> /+5V
- D18 pad 2: Net-(D17-DOUT) -> /Dout18
- D18 pad 3: /+5V -> GND
- D18 pad 4: unconnected-(D18-NC-Pad4) -> Net-(D17-DOUT)
- D19 pad 1: /Dout21 -> /+5V
- D19 pad 2: /Din19 -> /Dout21
- D19 pad 3: /+5V -> GND
- D19 pad 4: unconnected-(D19-NC-Pad4) -> /Din19
- D2 pad 1: Net-(D2-DOUT) -> /+5V
- D2 pad 2: /Dout1 -> Net-(D2-DOUT)
- D2 pad 3: /+5V -> GND
- D2 pad 4: unconnected-(D2-NC-Pad4) -> /Dout1
- D20 pad 1: Net-(D20-DOUT) -> /+5V
- D20 pad 2: /Dout21 -> Net-(D20-DOUT)
- D20 pad 3: /+5V -> GND
- D20 pad 4: unconnected-(D20-NC-Pad4) -> /Dout21
- D21 pad 1: Net-(D21-DOUT) -> /+5V
- D21 pad 2: Net-(D20-DOUT) -> Net-(D21-DOUT)
- D21 pad 3: /+5V -> GND
- D21 pad 4: unconnected-(D21-NC-Pad4) -> Net-(D20-DOUT)
- D22 pad 1: Net-(D22-DOUT) -> /+5V
- D22 pad 2: Net-(D21-DOUT) -> Net-(D22-DOUT)
- D22 pad 3: /+5V -> GND
- D22 pad 4: unconnected-(D22-NC-Pad4) -> Net-(D21-DOUT)
- D23 pad 1: Net-(D23-DOUT) -> /+5V
- D23 pad 2: Net-(D22-DOUT) -> Net-(D23-DOUT)
- D23 pad 3: /+5V -> GND
- D23 pad 4: unconnected-(D23-NC-Pad4) -> Net-(D22-DOUT)
- D24 pad 1: Net-(D24-DOUT) -> /+5V
- D24 pad 2: Net-(D23-DOUT) -> Net-(D24-DOUT)
- D24 pad 3: /+5V -> GND
- D24 pad 4: unconnected-(D24-NC-Pad4) -> Net-(D23-DOUT)
- D25 pad 1: Net-(D25-DOUT) -> /+5V
- D25 pad 2: Net-(D24-DOUT) -> Net-(D25-DOUT)
- D25 pad 3: /+5V -> GND
- D25 pad 4: unconnected-(D25-NC-Pad4) -> Net-(D24-DOUT)
- D26 pad 1: Net-(D26-DOUT) -> /+5V
- D26 pad 2: Net-(D25-DOUT) -> Net-(D26-DOUT)
- D26 pad 3: /+5V -> GND
- D26 pad 4: unconnected-(D26-NC-Pad4) -> Net-(D25-DOUT)
- D27 pad 1: /Dout27 -> /+5V
- D27 pad 2: Net-(D26-DOUT) -> /Dout27
- D27 pad 3: /+5V -> GND
- D27 pad 4: unconnected-(D27-NC-Pad4) -> Net-(D26-DOUT)
- D3 pad 1: Net-(D3-DOUT) -> /+5V
- D3 pad 2: Net-(D2-DOUT) -> Net-(D3-DOUT)
- D3 pad 3: /+5V -> GND
- D3 pad 4: unconnected-(D3-NC-Pad4) -> Net-(D2-DOUT)
- D4 pad 1: Net-(D4-DOUT) -> /+5V
- D4 pad 2: Net-(D3-DOUT) -> Net-(D4-DOUT)
- D4 pad 3: /+5V -> GND
- D4 pad 4: unconnected-(D4-NC-Pad4) -> Net-(D3-DOUT)
- D5 pad 1: Net-(D5-DOUT) -> /+5V
- D5 pad 2: Net-(D4-DOUT) -> Net-(D5-DOUT)
- D5 pad 3: /+5V -> GND
- D5 pad 4: unconnected-(D5-NC-Pad4) -> Net-(D4-DOUT)
- D6 pad 1: Net-(D6-DOUT) -> /+5V
- D6 pad 2: Net-(D5-DOUT) -> Net-(D6-DOUT)
- D6 pad 3: /+5V -> GND
- D6 pad 4: unconnected-(D6-NC-Pad4) -> Net-(D5-DOUT)
- D7 pad 1: Net-(D7-DOUT) -> /+5V
- D7 pad 2: Net-(D6-DOUT) -> Net-(D7-DOUT)
- D7 pad 3: /+5V -> GND
- D7 pad 4: unconnected-(D7-NC-Pad4) -> Net-(D6-DOUT)
- D8 pad 1: Net-(D8-DOUT) -> /+5V
- D8 pad 2: Net-(D7-DOUT) -> Net-(D8-DOUT)
- D8 pad 3: /+5V -> GND
- D8 pad 4: unconnected-(D8-NC-Pad4) -> Net-(D7-DOUT)
- D9 pad 1: /Dout9 -> /+5V
- D9 pad 2: Net-(D8-DOUT) -> /Dout9
- D9 pad 3: /+5V -> GND
- D9 pad 4: unconnected-(D9-NC-Pad4) -> Net-(D8-DOUT)
Routing:
- net GND: track 173.2 -> 312.4 mm
- net Net-(D7-DOUT): track 13.5 -> 7.87 mm
- net Net-(D16-DOUT): track 13.5 -> 7.87 mm
- net Net-(D25-DOUT): track 13.5 -> 7.87 mm
- net Net-(D6-DOUT): track 13.4 -> 7.87 mm
- net Net-(D5-DOUT): track 13.4 -> 7.87 mm
- net Net-(D8-DOUT): track 13.4 -> 7.87 mm
- net Net-(D20-DOUT): track 13.4 -> 7.87 mm
- net Net-(D17-DOUT): track 13.4 -> 7.87 mm
- net Net-(D14-DOUT): track 13.4 -> 7.87 mm
- net Net-(D11-DOUT): track 13.4 -> 7.87 mm
- net /Dout11: track 13.4 -> 7.87 mm
- net Net-(D3-DOUT): track 13.4 -> 7.87 mm
- net Net-(D21-DOUT): track 13.4 -> 7.87 mm
- net Net-(D2-DOUT): track 13.4 -> 7.87 mm
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Other:
- board text added: "locked"
