File: Hardware/TestingRig/TestingRig.kicad_sch (KiCad schematic)
At the start: 60 parts, among them J1 Conn_01x04_Pin, J2 Conn_01x04_Pin, J3 Conn_01x04_Pin, J4 Conn_01x04_Pin, J5 Conn_01x04_Pin, J6 Conn_01x04_Pin

Commit message: $1
Parts:
- D1, D10, D11, D12, D13, D14, D15, D16, D17, D18, D19, D2, D20, D21, D22, D23, D24, D25, D26, D27, D3, D4, D5, D6, D7, D8, D9: Extended (none) -> 1; Populate (none) -> Yes
- J1, J2, J3, J4, J5, J6: Populate (none) -> No
Changed lines of the file:
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@@
       (effects (font (size 1.27 1.27)) hide)
     )
+    (property "Extended" "1" (at 108.585 106.68 0)
+      (effects (font (size 1.27 1.27)) hide)
+    )
+    (property "Populate" "Yes" (at 108.585 106.68 0)
+      (effects (font (size 1.27 1.27)) hide)
+    )
     (pin "1")
     (pin "2")
@@
       (effects (font (size 1.27 1.27)) hide)
     )
+    (property "Extended" "1" (at 188.595 106.68 0)
+      (effects (font (size 1.27 1.27)) hide)
+    )
+    (property "Populate" "Yes" (at 188.595 106.68 0)
+      (effects (font (size 1.27 1.27)) hide)
+    )
     (pin "1")
     (pin "2")
@@
       (effects (font (size 1.27 1.27)) hide)
     )
+    (property "Extended" "1" (at 53.975 69.215 0)
+      (effects (font (size 1.27 1.27)) hide)
+    )
+    (property "Populate" "Yes" (at 53.975 69.215 0)
+      (effects (font (size 1.27 1.27)) hide)
+    )
     (pin "1")
     (pin "2")
@@
       (effects (font (size 1.27 1.27)) hide)
     )
+    (property "Extended" "1" (at 55.245 106.68 0)
+      (effects (font (size 1.27 1.27)) hide)
+    )
+    (property "Populate" "Yes" (at 55.245 106.68 0)
+      (effects (font (size 1.27 1.27)) hide)
+    )
     (pin "1")
     (pin "2")
@@
       (effects (font (size 1.27 1.27)) hide)
     )
+    (property "Extended" "1" (at 28.575 106.68 0)
+      (effects (font (size 1.27 1.27)) hide)
+    )
+    (property "Populate" "Yes" (at 28.575 106.68 0)
+      (effects (font (size 1.27 1.27)) hide)
+    )
     (pin "1")
     (pin "2")
@@
       (effects (font (size 1.27 1.27)) hide)
     )
+    (property "Extended" "1" (at 107.315 69.215 0)
+      (effects (font (size 1.27 1.27)) hide)
+    )
+    (property "Populate" "Yes" (at 107.315 69.215 0)
+      (effects (font (size 1.27 1.27)) hide)
+    )
     (pin "1")
     (pin "2")
@@
       (effects (font (size 1.27 1.27)) hide)
     )
+    (property "Extended" "1" (at 215.265 106.68 0)
+      (effects (font (size 1.27 1.27)) hide)
+    )
+    (property "Populate" "Yes" (at 215.265 106.68 0)
+      (effects (font (size 1.27 1.27)) hide)
+    )
     (pin "1")
     (pin "2")
@@
       (effects (font (size 1.27 1.27)) hide)
     )
+    (property "Extended" "1" (at 161.925 106.68 0)
+      (effects (font (size 1.27 1.27)) hide)
+    )
+    (property "Populate" "Yes" (at 161.925 106.68 0)
+      (effects (font (size 1.27 1.27)) hide)
+    )
     (pin "1")
     (pin "2")
@@
       (effects (font (size 1.27 1.27)) hide)
     )
+    (property "Extended" "1" (at 135.255 106.68 0)
+      (effects (font (size 1.27 1.27)) hide)
+    )
+    (property "Populate" "Yes" (at 135.255 106.68 0)
+      (effects (font (size 1.27 1.27)) hide)
+    )
     (pin "1")
     (pin "2")
@@
       (effects (font (size 1.27 1.27)) hide)
     )
+    (property "Extended" "1" (at 241.935 106.68 0)
+      (effects (font (size 1.27 1.27)) hide)
+    )
+    (property "Populate" "Yes" (at 241.935 106.68 0)
+      (effects (font (size 1.27 1.27)) hide)
+    )
     (pin "1")
     (pin "2")
@@
       (effects (font (size 1.27 1.27)) hide)
     )
+    (property "Extended" "1" (at 213.995 69.215 0)
+      (effects (font (size 1.27 1.27)) hide)
+    )
+    (property "Populate" "Yes" (at 213.995 69.215 0)
+      (effects (font (size 1.27 1.27)) hide)
+    )
     (pin "1")
     (pin "2")
@@
       (effects (font (size 1.27 1.27)) hide)
     )
+    (property "Extended" "1" (at 107.315 32.385 0)
+      (effects (font (size 1.27 1.27)) hide)
+    )
+    (property "Populate" "Yes" (at 107.315 32.385 0)
+      (effects (font (size 1.27 1.27)) hide)
+    )
     (pin "1")
     (pin "2")
@@
       (effects (font (size 1.27 1.27)) hide)
     )
+    (property "Extended" "1" (at 160.655 32.385 0)
+      (effects (font (size 1.27 1.27)) hide)
+    )
+    (property "Populate" "Yes" (at 160.655 32.385 0)
+      (effects (font (size 1.27 1.27)) hide)
+    )
     (pin "1")
     (pin "2")
@@
       (effects (font (size 1.27 1.27)))
     )
+    (property "Populate" "No" (at 226.06 135.89 0)
+      (effects (font (size 1.27 1.27)) hide)
+    )
     (pin "1")
     (pin "2")
@@
       (effects (font (size 1.27 1.27)))
     )
+    (property "Populate" "No" (at 245.745 135.255 0)
+      (effects (font (size 1.27 1.27)) hide)
+    )
     (pin "1")
     (pin "2")
@@
       (effects (font (size 1.27 1.27)) hide)
     )
+    (property "Extended" "1" (at 160.655 69.215 0)
+      (effects (font (size 1.27 1.27)) hide)
+    )
+    (property "Populate" "Yes" (at 160.655 69.215 0)
+      (effects (font (size 1.27 1.27)) hide)
+    )
     (pin "1")
     (pin "2")
@@
       (effects (font (size 1.27 1.27)) hide)
     )
+    (property "Extended" "1" (at 80.645 69.215 0)
+      (effects (font (size 1.27 1.27)) hide)
+    )
+    (property "Populate" "Yes" (at 80.645 69.215 0)
+      (effects (font (size 1.27 1.27)) hide)
+    )
     (pin "1")
     (pin "2")
@@
       (effects (font (size 1.27 1.27)) hide)
     )
+    (property "Extended" "1" (at 53.975 32.385 0)
+      (effects (font (size 1.27 1.27)) hide)
+    )
+    (property "Populate" "Yes" (at 53.975 32.385 0)
+      (effects (font (size 1.27 1.27)) hide)
+    )
     (pin "1")
     (pin "2")
@@
       (effects (font (size 1.27 1.27)))
     )
+    (property "Populate" "No" (at 210.185 135.89 0)
+      (effects (font (size 1.27 1.27)) hide)
+    )
     (pin "1")
     (pin "2")
@@
       (effects (font (size 1.27 1.27)) hide)
     )
+    (property "Extended" "1" (at 81.915 106.68 0)
+      (effects (font (size 1.27 1.27)) hide)
+    )
+    (property "Populate" "Yes" (at 81.915 106.68 0)
+      (effects (font (size 1.27 1.27)) hide)
+    )
     (pin "1")
     (pin "2")
@@
       (effects (font (size 1.27 1.27)) hide)
     )
+    (property "Extended" "1" (at 213.995 32.385 0)
+      (effects (font (size 1.27 1.27)) hide)
+    )
+    (property "Populate" "Yes" (at 213.995 32.385 0)
+      (effects (font (size 1.27 1.27)) hide)
+    )
     (pin "1")
     (pin "2")
@@
       (effects (font (size 1.27 1.27)) hide)
     )
+    (property "Extended" "1" (at 187.325 69.215 0)
+      (effects (font (size 1.27 1.27)) hide)
+    )
+    (property "Populate" "Yes" (at 187.325 69.215 0)
+      (effects (font (size 1.27 1.27)) hide)
+    )
     (pin "1")
     (pin "2")
@@
       (effects (font (size 1.27 1.27)) hide)
     )
+    (property "Extended" "1" (at 133.985 69.215 0)
+      (effects (font (size 1.27 1.27)) hide)
+    )
+    (property "Populate" "Yes" (at 133.985 69.215 0)
+      (effects (font (size 1.27 1.27)) hide)
+    )
     (pin "1")
     (pin "2")
@@
       (effects (font (size 1.27 1.27)) hide)
     )
+    (property "Extended" "1" (at 80.645 32.385 0)
+      (effects (font (size 1.27 1.27)) hide)
+    )
+    (property "Populate" "Yes" (at 80.645 32.385 0)
+      (effects (font (size 1.27 1.27)) hide)
+    )
     (pin "1")
     (pin "2")
@@
       (effects (font (size 1.27 1.27)))
     )
+    (property "Populate" "No" (at 261.62 135.255 0)
+      (effects (font (size 1.27 1.27)) hide)
+    )
     (pin "1")
     (pin "2")
@@
       (effects (font (size 1.27 1.27)))
     )
+    (property "Populate" "No" (at 175.895 135.89 0)
+      (effects (font (size 1.27 1.27)) hide)
+    )
     (pin "1")
     (pin "2")
@@
       (effects (font (size 1.27 1.27)) hide)
     )
+    (property "Extended" "1" (at 240.665 32.385 0)
+      (effects (font (size 1.27 1.27)) hide)
+    )
+    (property "Populate" "Yes" (at 240.665 32.385 0)
+      (effects (font (size 1.27 1.27)) hide)
+    )
     (pin "1")
     (pin "2")
@@
       (effects (font (size 1.27 1.27)) hide)
     )
+    (property "Extended" "1" (at 27.305 32.385 0)
+      (effects (font (size 1.27 1.27)) hide)
+    )
+    (property "Populate" "Yes" (at 27.305 32.385 0)
+      (effects (font (size 1.27 1.27)) hide)
+    )
     (pin "1")
     (pin "2")
@@
       (effects (font (size 1.27 1.27)))
     )
+    (property "Populate" "No" (at 191.77 135.89 0)
+      (effects (font (size 1.27 1.27)) hide)
+    )
     (pin "1")
     (pin "2")
@@
       (effects (font (size 1.27 1.27)) hide)
     )
+    (property "Extended" "1" (at 27.305 69.215 0)
+      (effects (font (size 1.27 1.27)) hide)
+    )
+    (property "Populate" "Yes" (at 27.305 69.215 0)
+      (effects (font (size 1.27 1.27)) hide)
+    )
     (pin "1")
     (pin "2")
@@
       (effects (font (size 1.27 1.27)) hide)
     )
+    (property "Extended" "1" (at 187.325 32.385 0)
+      (effects (font (size 1.27 1.27)) hide)
+    )
+    (property "Populate" "Yes" (at 187.325 32.385 0)
+      (effects (font (size 1.27 1.27)) hide)
+    )
     (pin "1")
     (pin "2")
@@
       (effects (font (size 1.27 1.27)) hide)
     )
+    (property "Extended" "1" (at 240.665 69.215 0)
+      (effects (font (size 1.27 1.27)) hide)
+    )
+    (property "Populate" "Yes" (at 240.665 69.215 0)
+      (effects (font (size 1.27 1.27)) hide)
+    )
     (pin "1")
     (pin "2")
@@
       (effects (font (size 1.27 1.27)) hide)
     )
+    (property "Extended" "1" (at 133.985 32.385 0)
+      (effects (font (size 1.27 1.27)) hide)
+    )
+    (property "Populate" "Yes" (at 133.985 32.385 0)
+      (effects (font (size 1.27 1.27)) hide)
+    )

Commit message: message
Parts:
- D1, D10, D11, D12, D13, D14, D15, D16, D17, D18, D19, D2, D20, D21, D22, D23, D24, D25, D26, D27, D3, D4, D5, D6, D7, D8, D9: footprint LED_SMD:LED_WS2812_PLCC6_5.0x5.0mm_P1.6mm -> LED_SMD:LED_WS2812B_PLCC4_5.0x5.0mm_P3.2mm; symbol LED:WS2812 -> LED:WS2812B
Connections:
- net +5V: now also D1.1 (VDD), D10.1 (VDD), D11.1 (VDD), D12.1 (VDD), D13.1 (VDD), D14.1 (VDD), D15.1 (VDD), D16.1 (VDD), D17.1 (VDD), D18.1 (VDD), D19.1 (VDD), D2.1 (VDD), D20.1 (VDD), D21.1 (VDD), D22.1 (VDD), D23.1 (VDD), D24.1 (VDD), D25.1 (VDD), D26.1 (VDD), D27.1 (VDD), D3.1 (VDD), D4.1 (VDD), D5.1 (VDD), D6.1 (VDD), D7.1 (VDD), D8.1 (VDD), D9.1 (VDD); no longer D1.3 (VCC), D1.5 (VDD), D10.3 (VCC), D10.5 (VDD), D11.3 (VCC), D11.5 (VDD), D12.3 (VCC), D12.5 (VDD), D13.3 (VCC), D13.5 (VDD), D14.3 (VCC), D14.5 (VDD), D15.3 (VCC), D15.5 (VDD), D16.3 (VCC), D16.5 (VDD), D17.3 (VCC), D17.5 (VDD), D18.3 (VCC), D18.5 (VDD), D19.3 (VCC), D19.5 (VDD), D2.3 (VCC), D2.5 (VDD), D20.3 (VCC), D20.5 (VDD), D21.3 (VCC), D21.5 (VDD), D22.3 (VCC), D22.5 (VDD), D23.3 (VCC), D23.5 (VDD), D24.3 (VCC), D24.5 (VDD), D25.3 (VCC), D25.5 (VDD), D26.3 (VCC), D26.5 (VDD), D27.3 (VCC), D27.5 (VDD), D3.3 (VCC), D3.5 (VDD), D4.3 (VCC), D4.5 (VDD), D5.3 (VCC), D5.5 (VDD), D6.3 (VCC), D6.5 (VDD), D7.3 (VCC), D7.5 (VDD), D8.3 (VCC), D8.5 (VDD), D9.3 (VCC), D9.5 (VDD)
- net Din1: now also D1.4 (DIN); no longer D1.2 (DIN)
- net Din10: now also D10.4 (DIN); no longer D10.2 (DIN)
- net Din19: now also D19.4 (DIN); no longer D19.2 (DIN)
- net Dout1: now also D1.2 (DOUT), D2.4 (DIN); no longer D1.1 (DOUT), D2.2 (DIN)
- net Dout11: now also D10.2 (DOUT), D11.4 (DIN); no longer D10.1 (DOUT), D11.2 (DIN)
- net Dout18: now also D18.2 (DOUT); no longer D18.1 (DOUT)
- net Dout21: now also D19.2 (DOUT), D20.4 (DIN); no longer D19.1 (DOUT), D20.2 (DIN)
- net Dout27: now also D27.2 (DOUT); no longer D27.1 (DOUT)
- net Dout9: now also D9.2 (DOUT); no longer D9.1 (DOUT)
- net GND: now also D1.3 (VSS), D10.3 (VSS), D11.3 (VSS), D12.3 (VSS), D13.3 (VSS), D14.3 (VSS), D15.3 (VSS), D16.3 (VSS), D17.3 (VSS), D18.3 (VSS), D19.3 (VSS), D2.3 (VSS), D20.3 (VSS), D21.3 (VSS), D22.3 (VSS), D23.3 (VSS), D24.3 (VSS), D25.3 (VSS), D26.3 (VSS), D27.3 (VSS), D3.3 (VSS), D4.3 (VSS), D5.3 (VSS), D6.3 (VSS), D7.3 (VSS), D8.3 (VSS), D9.3 (VSS); no longer D1.6 (VSS), D10.6 (VSS), D11.6 (VSS), D12.6 (VSS), D13.6 (VSS), D14.6 (VSS), D15.6 (VSS), D16.6 (VSS), D17.6 (VSS), D18.6 (VSS), D19.6 (VSS), D2.6 (VSS), D20.6 (VSS), D21.6 (VSS), D22.6 (VSS), D23.6 (VSS), D24.6 (VSS), D25.6 (VSS), D26.6 (VSS), D27.6 (VSS), D3.6 (VSS), D4.6 (VSS), D5.6 (VSS), D6.6 (VSS), D7.6 (VSS), D8.6 (VSS), D9.6 (VSS)
- net at D23.2 (DOUT): now also D24.4 (DIN); no longer D22.1 (DOUT)
- net at D22.2 (DOUT): now also D23.4 (DIN); no longer D21.1 (DOUT)
- net at D22.4 (DIN): now also D21.2 (DOUT)
- net at D26.2 (DOUT): now also D27.4 (DIN); no longer D25.1 (DOUT)
- net at D25.2 (DOUT): now also D26.4 (DIN); no longer D24.1 (DOUT)
- net at D25.4 (DIN): now also D24.2 (DOUT)
- net at D12.2 (DOUT): now also D13.4 (DIN); no longer D11.1 (DOUT)
- net at D14.2 (DOUT): now also D15.4 (DIN); no longer D13.1 (DOUT)
- net at D13.2 (DOUT): now also D14.4 (DIN); no longer D12.1 (DOUT)
- net at D17.2 (DOUT): now also D18.4 (DIN); no longer D16.1 (DOUT)
- net at D17.4 (DIN): now also D16.2 (DOUT)
- net at D5.2 (DOUT): now also D6.4 (DIN); no longer D4.1 (DOUT)
- net at D4.2 (DOUT): now also D5.4 (DIN); no longer D3.1 (DOUT)
- net at D4.4 (DIN): now also D3.2 (DOUT)
- net at D7.2 (DOUT): now also D8.4 (DIN); no longer D6.1 (DOUT)
- net at D6.2 (DOUT): now also D7.4 (DIN); no longer D5.1 (DOUT)
- net at D15.2 (DOUT): now also D16.4 (DIN); no longer D14.1 (DOUT)
- net at D12.4 (DIN): now also D11.2 (DOUT)
- net at D21.4 (DIN): now also D20.2 (DOUT)
- net at D8.2 (DOUT): now also D9.4 (DIN); no longer D7.1 (DOUT)
- net at D3.4 (DIN): now also D2.2 (DOUT)
