File: Hardware/LightSensor/LightSensor.kicad_pcb (KiCad board)
At the start: 2 copper layers, 18 x 13 mm, 7 parts, among them J1 Conn_01x04_Pin, U1 VEML6040

Commit message: $1
Parts:
- added C2: 100n, Capacitor_SMD:C_0603_1608Metric, F.Cu at (226.9, 110.8)
- added R3: 4.7k, Resistor_SMD:R_0603_1608Metric, F.Cu at (209.8, 108.1)
- added U2: TMP116xxDRV, Package_SON:WSON-6-1EP_2x2mm_P0.65mm_EP1x1.6mm, F.Cu at (226.1, 113.7)
- J1: footprint Connector_PinHeader_2.54mm:PinHeader_1x04_P2.54mm_Vertical -> Connector_PinHeader_2.54mm:PinHeader_1x05_P2.54mm_Vertical
- moved G*** 13.7 mm to (224.6, 104.5)
- moved R1 9.89 mm to (209.8, 113.1)
- moved G*** 6.83 mm to (213.5, 104.0)
- moved R2 6.76 mm to (209.8, 110.6), turned to 0 degrees
- moved C1 5.36 mm to (221.5, 115.6), turned to 180 degrees
- moved J1 3.63 mm to (213.8, 108.0)
- moved U1 1.59 mm to (221.8, 113.2)
Connections:
- J1 pad 3: /+3.3V -> /ALERT
- J1 pad 4: GND -> /+3.3V
- R1 pad 2: /SDA -> /ALERT
Routing:
- net /+3.3V: track 12.9 -> 36.3 mm, vias 0 -> 1
- net /ALERT: track 0.00 -> 19.5 mm, vias 0 -> 2
- net /SCL: track 9.08 -> 20.8 mm, vias 0 -> 2
- net /SDA: track 15.8 -> 16.9 mm
- net (no net): vias 0 -> 2
Other:
- board size 18 x 13 mm -> 30.5 x 23 mm

Commit message: message
Parts:
- U2: value TMP116xxDRV -> TMP117xxDRV
- moved C2 4.16 mm to (230.0, 113.5)
- moved C1 1.14 mm to (220.7, 116.4), turned to 90 degrees
- moved U2 0.36 mm to (226.4, 113.5), turned to 0 degrees
Routing:
- net /SDA: track 16.9 -> 31.5 mm, vias 0 -> 1
- net /SCL: track 20.8 -> 26.3 mm, vias 2 -> 1
- net /+3.3V: track 36.3 -> 40.4 mm
- net /ALERT: track 19.5 -> 16.2 mm
- net GND: track 0.00 -> 2.55 mm, vias 0 -> 2
Other:
- board text added: "ALERT"

Commit message: message
Other:
- board text added: "V1"
Changed lines of the file:
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@@
     (effects (font (size 0.8 0.8) (thickness 0.15)) (justify left bottom mirror))
   )
-  (gr_text "VEML6040 \nBreakout Board" (at 236 117.1 90) (layer "F.SilkS")
+  (gr_text "VEML6040 \nBreakout Board" (at 236 117.5 90) (layer "F.SilkS")
+    (effects (font (size 0.8 0.8) (thickness 0.15)) (justify left bottom))
+  )
+  (gr_text "V1" (at 207.9 123.4) (layer "F.SilkS")
     (effects (font (size 0.8 0.8) (thickness 0.15)) (justify left bottom))
   )
@@
     (pts (xy 237.25 122.7) (xy 206.75 122.7))
     (height -7.6)
-    (gr_text "30.5000 mm" (at 222 129.15) (layer "User.1")
+    (gr_text "30,5000 mm" (at 222 129.15) (layer "User.1")
       (effects (font (size 1 1) (thickness 0.15)))
     )
@@
     (pts (xy 235 103.6) (xy 235 122.6))
     (height -9)
-    (gr_text locked "19.0000 mm" (at 242.85 113.1 90) (layer "User.1")
+    (gr_text locked "19,0000 mm" (at 242.85 113.1 90) (layer "User.1")
       (effects (font (size 1 1) (thickness 0.15)))
     )
@@
     (pts (xy 235 103.6) (xy 237.2 103.6))
     (height -8.8)
-    (gr_text "2.2000 mm" (at 236.1 93.65) (layer "User.1")
+    (gr_text "2,2000 mm" (at 236.1 93.65) (layer "User.1")
       (effects (font (size 1 1) (thickness 0.15)))
     )
@@
     (pts (xy 237.25 103.7) (xy 237.25 113.2))
     (height -14.15)
-    (gr_text "9.5000 mm" (at 250.25 108.45 90) (layer "User.1")
+    (gr_text "9,5000 mm" (at 250.25 108.45 90) (layer "User.1")
       (effects (font (size 1 1) (thickness 0.15)))
     )
@@
     (pts (xy 206.75 103.7) (xy 237.25 103.7))
     (height -11.2)
-    (gr_text "30.5000 mm" (at 222 91.35) (layer "User.1")
+    (gr_text "30,5000 mm" (at 222 91.35) (layer "User.1")
       (effects (font (size 1 1) (thickness 0.15)))
     )
@@
     (pts (xy 235.25 101.7) (xy 235.25 124.7))
     (height -12.45)
-    (gr_text "23.0000 mm" (at 246.55 113.2 90) (layer "User.1")
+    (gr_text "23,0000 mm" (at 246.55 113.2 90) (layer "User.1")
       (effects (font (size 1 1) (thickness 0.15)))
     )
