File: Hardware/LightSensor/LightSensor.kicad_pcb (KiCad board)
At the start: 2 copper layers, 30.5 x 23 mm, 10 parts, among them J1 Conn_01x04_Pin, U1 VEML6040, U2 TMP117xxDRV

Commit message: $1
Parts:
- added G***: LOGO, LOGO, F.Cu at (227.0, 121.8)
- added G***: LOGO, LOGO, F.Cu at (215.9, 122.3)
- added J2: Conn_01x04_Pin, uct:conn_01x05_2.54_SMD_5mm, F.Cu at (222.0, 104.6)
- moved J1 0.30 mm to (213.5, 108.0)
Routing:
- net /ALERT: track 16.2 -> 28.5 mm, vias 2 -> 3
- net /+3.3V: track 40.4 -> 51.2 mm
- net /SCL: track 26.3 -> 34.5 mm
- net /SDA: track 31.5 -> 34.4 mm
Other:
- board text added: "AL"
