File: Hardware/LightSensor/LightSensor.kicad_sch (KiCad schematic)
At the start: 5 parts, among them J1 Conn_01x04_Pin, U1 VEML6040

Commit message: $1
Parts:
- added C2: 100n, Capacitor_SMD:C_0603_1608Metric, symbol Device:C_Small
- added D1: WS2812, LED_SMD:LED_WS2812_PLCC6_5.0x5.0mm_P1.6mm, symbol LED:WS2812
Connections:
- new net +5V: C2.2, D1.3 (VCC), D1.5 (VDD)
- new net Din: D1.2 (DIN)
- new net Dout: D1.1 (DOUT)
- new net GND1: C2.1, D1.6 (VSS)
Other:
- note added: "VEML6040 Ambient Light Sensor"
- moved on the sheet: C2, J1, R1, R2, U1

Commit message: $1
Parts:
- removed D1: WS2812, LED_SMD:LED_WS2812_PLCC6_5.0x5.0mm_P1.6mm, symbol LED:WS2812
- added R3: 4.7k, Resistor_SMD:R_0603_1608Metric, symbol Device:R_US
- added U2: TMP116xxDRV, Package_SON:WSON-6-1EP_2x2mm_P0.65mm_EP1x1.6mm, symbol Sensor_Temperature:TMP116xxDRV
- J1: footprint Connector_PinHeader_2.54mm:PinHeader_1x04_P2.54mm_Vertical -> Connector_PinHeader_2.54mm:PinHeader_1x05_P2.54mm_Vertical; symbol Connector:Conn_01x04_Pin -> Connector:Conn_01x05_Pin
Connections:
- net +5V is gone; now on net +3.3V: C2.2
- net GND1 is gone; now on net GND: C2.1
- net +3.3V: now also J1.4 (Pin_4), R3.1, U2.5 (V+); no longer J1.3 (Pin_3)
- net GND: now also J1.5 (Pin_5), U2.2 (GND), U2.4 (ADD0); no longer J1.4 (Pin_4)
- net SCL: now also U2.1 (SCL)
- net SDA: now also R3.2, U2.6 (SDA); no longer R1.2
- new net ALERT: J1.3 (Pin_3), R1.2, U2.3 (ALERT)
Other:
- note added: "Pull-up resistors, input cap, output pins"
- note added: "Temperature Sensor"
- moved on the sheet: C2, U1

Commit message: message
Parts:
- removed U2: TMP116xxDRV, Package_SON:WSON-6-1EP_2x2mm_P0.65mm_EP1x1.6mm, symbol Sensor_Temperature:TMP116xxDRV
- added U2: TMP117xxDRV, Package_SON:WSON-6-1EP_2x2mm_P0.65mm_EP1x1.6mm, symbol Sensor_Temperature:TMP117xxDRV
Connections:
- net +3.3V: now also U2.5 (V+)
- net ALERT: now also U2.3 (ALERT)
- net GND: now also U2.2 (GND), U2.4 (ADD0)
- net SCL: now also U2.1 (SCL)
- net SDA: now also U2.6 (SDA)
Changed lines of the file:
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@@
+    )
+  )
+  (symbol (lib_id "Sensor_Temperature:TMP117xxDRV") (at 215.9 142.24 0) (unit 1)
+    (in_bom yes) (on_board yes) (dnp no)
+    (property "Reference" "U2" (at 231.14 146.05 0)
+      (effects (font (size 1.27 1.27)))
+    )
+    (property "Value" "TMP117xxDRV" (at 231.14 148.59 0)
+      (effects (font (size 1.27 1.27)))
+    )
+    (property "Footprint" "Package_SON:WSON-6-1EP_2x2mm_P0.65mm_EP1x1.6mm" (at 217.17 151.13 0)
+      (effects (font (size 1.27 1.27)) (justify left) hide)
+    )
+    (property "Datasheet" "https://www.ti.com/lit/ds/symlink/tmp117.pdf" (at 217.17 153.67 0)
+      (effects (font (size 1.27 1.27)) (justify left) hide)
+    )
+    (property "Extended" "1" (at 215.9 142.24 0)
+      (effects (font (size 1.27 1.27)) hide)
+    )
+    (property "LCSC" "C699536" (at 215.9 142.24 0)
+      (effects (font (size 1.27 1.27)) hide)
+    )
+    (property "Populate" "Yes" (at 215.9 142.24 0)
+      (effects (font (size 1.27 1.27)) hide)
+    )
+    (pin "1")
+    (pin "2")
+    (pin "3")
+    (pin "4")
+    (pin "5")
+    (pin "6")
+    (instances
+      (project "LightSensor"
+        (path "/8985338b-1403-4fdb-a4a7-da7f590a3346"
+          (reference "U2") (unit 1)
+        )
+      )
     )
   )
@@
         )
       )
-    )
-  )
-  (symbol (lib_id "Sensor_Temperature:TMP116xxDRV") (at 215.9 142.24 0) (unit 1)
-    (in_bom yes) (on_board yes) (dnp no)
-    (property "Reference" "U2" (at 231.14 146.685 0)
-      (effects (font (size 1.27 1.27)))
-    )
-    (property "Value" "TMP116xxDRV" (at 231.14 149.225 0)
-      (effects (font (size 1.27 1.27)))
-    )
-    (property "Footprint" "Package_SON:WSON-6-1EP_2x2mm_P0.65mm_EP1x1.6mm" (at 217.17 151.13 0)
-      (effects (font (size 1.27 1.27)) (justify left) hide)
-    )
-    (property "Datasheet" "https://www.ti.com/lit/ds/symlink/tmp116.pdf" (at 217.17 153.67 0)
-      (effects (font (size 1.27 1.27)) (justify left) hide)
-    )
-    (property "LCSC" "C2691433" (at 215.9 142.24 0)
-      (effects (font (size 1.27 1.27)) hide)
-    )
-    (pin "1")
-    (pin "2")
-    (pin "3")
-    (pin "4")
-    (pin "5")
-    (pin "6")
-    (instances
-      (project "LightSensor"
-        (path "/8985338b-1403-4fdb-a4a7-da7f590a3346"
-          (reference "U2") (unit 1)
-        )
-      )

Commit message: message
Parts:
- added J2: Conn_01x05_Pin, symbol Connector:Conn_01x05_Pin
Connections:
- net +3.3V: now also J2.4 (Pin_4)
- net ALERT: now also J2.3 (Pin_3)
- net GND: now also J2.5 (Pin_5)
- net SCL: now also J2.2 (Pin_2)
- net SDA: now also J2.1 (Pin_1)
Changed lines of the file:
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@@
+    (stroke (width 0) (type default))
+  )
+  (wire (pts (xy 180.975 99.695) (xy 175.26 99.695))
     (stroke (width 0) (type default))
   )
@@
     (stroke (width 0) (type default))
   )
+  (wire (pts (xy 176.53 107.315) (xy 175.26 107.315))
+    (stroke (width 0) (type default))
+  )
   (wire (pts (xy 205.74 144.78) (xy 205.74 154.305))
     (stroke (width 0) (type default))
@@
     (stroke (width 0) (type default))
   )
+  (wire (pts (xy 180.975 97.155) (xy 175.26 97.155))
+    (stroke (width 0) (type default))
+  )
   (wire (pts (xy 269.24 112.395) (xy 261.62 112.395))
     (stroke (width 0) (type default))
@@
     (stroke (width 0) (type default))
   )
+  (wire (pts (xy 176.53 104.775) (xy 175.26 104.775))
+    (stroke (width 0) (type default))
+  )
   (wire (pts (xy 215.9 154.305) (xy 215.9 156.21))
+    (stroke (width 0) (type default))
+  )
+  (wire (pts (xy 180.975 102.235) (xy 175.26 102.235))
     (stroke (width 0) (type default))
   )
@@
     (effects (font (size 1.27 1.27)) (justify left bottom))
   )
+  (label "+3.3V" (at 176.53 104.775 0) (fields_autoplaced)
+    (effects (font (size 1.27 1.27)) (justify left bottom))
+  )
+  (label "SCL" (at 180.975 99.695 0) (fields_autoplaced)
+    (effects (font (size 1.27 1.27)) (justify left bottom))
+  )
   (label "ALERT" (at 232.41 137.16 180) (fields_autoplaced)
     (effects (font (size 1.27 1.27)) (justify right bottom))
@@
   )
   (label "SDA" (at 200.025 137.16 0) (fields_autoplaced)
+    (effects (font (size 1.27 1.27)) (justify left bottom))
+  )
+  (label "ALERT" (at 180.975 102.235 0) (fields_autoplaced)
+    (effects (font (size 1.27 1.27)) (justify left bottom))
+  )
+  (label "SDA" (at 180.975 97.155 0) (fields_autoplaced)
     (effects (font (size 1.27 1.27)) (justify left bottom))
   )
@@
     )
   )
+  (symbol (lib_id "Connector:Conn_01x05_Pin") (at 170.18 102.235 0) (unit 1)
+    (in_bom yes) (on_board yes) (dnp no) (fields_autoplaced)
+    (property "Reference" "J2" (at 170.815 93.345 0)
+      (effects (font (size 1.27 1.27)))
+    )
+    (property "Value" "Conn_01x05_Pin" (at 170.815 95.885 0)
+      (effects (font (size 1.27 1.27)))
+    )
+    (property "Footprint" "" (at 170.18 102.235 0)
+      (effects (font (size 1.27 1.27)) hide)
+    )
+    (property "Datasheet" "~" (at 170.18 102.235 0)
+      (effects (font (size 1.27 1.27)) hide)
+    )
+    (pin "1")
+    (pin "2")
+    (pin "3")
+    (pin "4")
+    (pin "5")
+    (instances
+      (project "LightSensor"
+        (path "/8985338b-1403-4fdb-a4a7-da7f590a3346"
+          (reference "J2") (unit 1)
+        )
+      )
+    )
+  )
   (symbol (lib_id "Connector:Conn_01x05_Pin") (at 196.85 104.14 0) (unit 1)
     (in_bom yes) (on_board yes) (dnp no)
@@
         )
       )
+    )
+  )
+  (symbol (lib_id "power:GND") (at 176.53 107.315 0) (unit 1)
+    (in_bom yes) (on_board yes) (dnp no) (fields_autoplaced)
+    (property "Reference" "#PWR05" (at 176.53 113.665 0)
+      (effects (font (size 1.27 1.27)) hide)
+    )
+    (property "Value" "GND" (at 176.53 111.76 0)
+      (effects (font (size 1.27 1.27)))
+    )
+    (property "Footprint" "" (at 176.53 107.315 0)
+      (effects (font (size 1.27 1.27)) hide)
+    )
+    (property "Datasheet" "" (at 176.53 107.315 0)
+      (effects (font (size 1.27 1.27)) hide)
+    )
+    (pin "1")
+    (instances
+      (project "LightSensor"
+        (path "/8985338b-1403-4fdb-a4a7-da7f590a3346"
+          (reference "#PWR05") (unit 1)
+        )
+      )
