File: Hardware/LightSensor/LightSensor.kicad_sch (KiCad schematic)
At the start: 8 parts, among them J1 Conn_01x04_Pin, U1 VEML6040, U2 TMP117xxDRV

Commit message: $1
Parts:
- added J2: Conn_01x04_Pin, uct:conn_01x05_2.54_SMD_5mm, symbol Connector:Conn_01x05_Pin
Connections:
- net +3.3V: now also J2.4 (Pin_4)
- net ALERT: now also J2.3 (Pin_3)
- net GND: now also J2.5 (Pin_5)
- net SCL: now also J2.2 (Pin_2)
- net SDA: now also J2.1 (Pin_1)
Changed lines of the file:
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@@
+    (stroke (width 0) (type default))
+  )
+  (wire (pts (xy 178.435 109.22) (xy 177.165 109.22))
     (stroke (width 0) (type default))
   )
@@
     (stroke (width 0) (type default))
   )
+  (wire (pts (xy 182.88 99.06) (xy 177.165 99.06))
+    (stroke (width 0) (type default))
+  )
   (wire (pts (xy 203.2 109.22) (xy 201.93 109.22))
     (stroke (width 0) (type default))
@@
     (stroke (width 0) (type default))
   )
+  (wire (pts (xy 178.435 106.68) (xy 177.165 106.68))
+    (stroke (width 0) (type default))
+  )
   (wire (pts (xy 261.62 104.14) (xy 269.24 104.14))
     (stroke (width 0) (type default))
@@
     (stroke (width 0) (type default))
   )
+  (wire (pts (xy 182.88 101.6) (xy 177.165 101.6))
+    (stroke (width 0) (type default))
+  )
   (wire (pts (xy 217.805 106.68) (xy 217.805 112.395))
     (stroke (width 0) (type default))
@@
     (stroke (width 0) (type default))
   )
+  (wire (pts (xy 182.88 104.14) (xy 177.165 104.14))
+    (stroke (width 0) (type default))
+  )
   (wire (pts (xy 205.74 154.305) (xy 215.9 154.305))
     (stroke (width 0) (type default))
@@
     (fill (type none))
   )
-  (rectangle (start 193.04 83.185) (end 273.05 121.92)
+  (rectangle (start 168.275 83.185) (end 273.05 121.92)
     (stroke (width 0) (type default))
     (fill (type none))
@@
     (effects (font (size 1.27 1.27)) (justify left bottom))
   )
+  (label "SCL" (at 182.88 101.6 0) (fields_autoplaced)
+    (effects (font (size 1.27 1.27)) (justify left bottom))
+  )
   (label "SDA" (at 245.11 96.52 0) (fields_autoplaced)
     (effects (font (size 1.27 1.27)) (justify left bottom))
@@
   )
   (label "ALERT" (at 245.11 112.395 0) (fields_autoplaced)
+    (effects (font (size 1.27 1.27)) (justify left bottom))
+  )
+  (label "ALERT" (at 182.88 104.14 0) (fields_autoplaced)
     (effects (font (size 1.27 1.27)) (justify left bottom))
   )
@@
     (effects (font (size 1.27 1.27)) (justify left bottom))
   )
+  (label "+3.3V" (at 178.435 106.68 0) (fields_autoplaced)
+    (effects (font (size 1.27 1.27)) (justify left bottom))
+  )
   (label "SDA" (at 200.025 137.16 0) (fields_autoplaced)
+    (effects (font (size 1.27 1.27)) (justify left bottom))
+  )
+  (label "SDA" (at 182.88 99.06 0) (fields_autoplaced)
     (effects (font (size 1.27 1.27)) (justify left bottom))
   )
@@
         (path "/8985338b-1403-4fdb-a4a7-da7f590a3346"
           (reference "#PWR06") (unit 1)
+        )
+      )
+    )
+  )
+  (symbol (lib_id "Connector:Conn_01x05_Pin") (at 172.085 104.14 0) (unit 1)
+    (in_bom yes) (on_board yes) (dnp no)
+    (property "Reference" "J2" (at 172.72 97.155 0)
+      (effects (font (size 1.27 1.27)))
+    )
+    (property "Value" "Conn_01x04_Pin" (at 176.53 97.79 0)
+      (effects (font (size 1.27 1.27)) hide)
+    )
+    (property "Footprint" "uct:conn_01x05_2.54_SMD_5mm" (at 172.085 104.14 0)
+      (effects (font (size 1.27 1.27)) hide)
+    )
+    (property "Datasheet" "~" (at 172.085 104.14 0)
+      (effects (font (size 1.27 1.27)) hide)
+    )
+    (property "LCSC" "" (at 172.085 104.14 0)
+      (effects (font (size 1.27 1.27)))
+    )
+    (property "Populate" "No" (at 172.085 104.14 0)
+      (effects (font (size 1.27 1.27)) hide)
+    )
+    (pin "1")
+    (pin "2")
+    (pin "3")
+    (pin "4")
+    (pin "5")
+    (instances
+      (project "LightSensor"
+        (path "/8985338b-1403-4fdb-a4a7-da7f590a3346"
+          (reference "J2") (unit 1)
         )
       )
@@
         )
       )
+    )
+  )
+  (symbol (lib_id "power:GND") (at 178.435 109.22 0) (unit 1)
+    (in_bom yes) (on_board yes) (dnp no) (fields_autoplaced)
+    (property "Reference" "#PWR05" (at 178.435 115.57 0)
+      (effects (font (size 1.27 1.27)) hide)
+    )
+    (property "Value" "GND" (at 178.435 113.665 0)
+      (effects (font (size 1.27 1.27)))
+    )
+    (property "Footprint" "" (at 178.435 109.22 0)
+      (effects (font (size 1.27 1.27)) hide)
+    )
+    (property "Datasheet" "" (at 178.435 109.22 0)
+      (effects (font (size 1.27 1.27)) hide)
+    )
+    (pin "1")
+    (instances
+      (project "LightSensor"
+        (path "/8985338b-1403-4fdb-a4a7-da7f590a3346"
+          (reference "#PWR05") (unit 1)
+        )
+      )
