File: Hardware/LightSensor.kicad_pcb (KiCad board)
At the start: 2 copper layers, 30.5 x 23 mm, 13 parts, among them J1 Conn_01x04_Pin, J2 Conn_01x04_Pin, U1 VEML6040, U2 TMP117xxDRV

Commit message: $1
Parts:
- moved C1 13.1 mm to (220.7, 116.4), turned to 90 degrees
- moved U1 12.2 mm to (221.8, 113.2)
- moved U2 1.03 mm to (226.4, 113.5)
- moved C2 0.13 mm to (230.0, 113.5)
Routing:
- net /ALERT: track 24.1 -> 28.5 mm, vias 2 -> 3
- net /+3.3V: track 48.7 -> 51.2 mm, vias 2 -> 1
- net /SCL: track 32.2 -> 34.5 mm, vias 0 -> 1
- net /SDA: track 36.1 -> 34.4 mm, vias 3 -> 1
- net GND: track 3.49 -> 2.55 mm, vias 3 -> 2
